File: PicoRubyMacroPad_PCB/PicoRubyMacroPad.sch (KiCad schematic (older format))
At the start: 29 parts, among them SW1 SW_Push, SW10 SW_Push, SW11 SW_Push, SW2 SW_Push, SW3 SW_Push, SW4 SW_Push, SW5 SW_Push, SW6 SW_Push, SW7 SW_Push, SW8 SW_Push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

Commit message: A diode added for SW11
Parts:
- added D11: D, kbd:D3_TH_SMD_v2, symbol Device:D
Connections:
- net R3: now also D11.1 (K); no longer SW11.1
- new net: D11.2 (A), SW11.1
Changed lines of the file:
@@
 Text GLabel 4375 2725 0    50   Input ~ 0
 R2
-Text GLabel 4375 3150 0    50   Input ~ 0
+Text GLabel 4375 3450 0    50   Input ~ 0
 R3
 Wire Wire Line
@@
 NoConn ~ 2825 1450
 Wire Wire Line
-	4375 3150 4650 3150
+	4375 3450 4650 3450
+$Comp
+L Device:D D11
+U 1 1 61AC63BF
+P 4650 3300
+F 0 "D11" V 4696 3220 50  0000 R CNN
+F 1 "D" V 4605 3220 50  0000 R CNN
+F 2 "kbd:D3_TH_SMD_v2" H 4650 3300 50  0001 C CNN
+F 3 "~" H 4650 3300 50  0001 C CNN
+	1    4650 3300
+	0    -1   -1   0
+$EndComp
 $EndSCHEMATC
